File: design-files/nabu-usb-keyboard.kicad_pcb (KiCad board)
At the start: 2 copper layers, 55.2 x 71.8 mm, 16 parts, among them J1 Console UART header, J2 Debug Event Header, J3 DIN-6, J4 9V input, Q1 SiHLU110-GE3, U1 74LVC245, U2 Pico, U3 SN75176AP

Commit message: Finalize the first prototype PCB.
Parts:
- removed J4: 9V input, Connector_BarrelJack:BarrelJack_CUI_PJ-102AH_Horizontal
- added C3: 1nF, Capacitor_THT:C_Disc_D6.0mm_W4.4mm_P5.00mm, F.Cu at (157.5, 121.9)
- added C4: 1nF, Capacitor_THT:C_Disc_D6.0mm_W4.4mm_P5.00mm, F.Cu at (157.5, 127.6)
- added D1: 1N4001, Diode_THT:D_DO-41_SOD81_P10.16mm_Horizontal, F.Cu at (158.1, 114.9)
- added R2: 180, Resistor_THT:R_Axial_DIN0207_L6.3mm_D2.5mm_P2.54mm_Vertical, F.Cu at (165.1, 125.7)
- added REF**: OSHW-Logo2_7.3x6mm_SilkScreen, Symbol:OSHW-Logo2_7.3x6mm_SilkScreen, F.Cu at (125.1, 124.5)
- C1, C2: footprint Capacitor_THT:C_Disc_D5.0mm_W2.5mm_P5.00mm -> Capacitor_THT:C_Disc_D6.0mm_W4.4mm_P5.00mm
- J2: value Debug Event Header -> DIN-6; footprint Connector_PinHeader_2.54mm:PinHeader_1x03_P2.54mm_Vertical -> jrt-Connectors:Jack_DIN-6_CLIFF_FC680806
- J3: value DIN-6 -> 9V input; footprint Connector_PinHeader_2.54mm:PinHeader_1x06_P2.54mm_Horizontal -> jrt-Connectors:Kobiconn_163-179PH-EX-5_5-2_1mm-1_5A
- Q1: value SiHLU110-GE3 -> IRLU110PBF
- R1: footprint Resistor_THT:R_Axial_DIN0204_L3.6mm_D1.6mm_P5.08mm_Horizontal -> Resistor_THT:R_Axial_DIN0207_L6.3mm_D2.5mm_P7.62mm_Horizontal
- moved J3 58.2 mm to (159.4, 62.5), turned to 0 degrees
- moved J2 28.7 mm to (144.1, 133.7), turned to 180 degrees
- moved R1 1.42 mm to (137.8, 112.4)
- moved U3 1.42 mm to (120.7, 108.0)
- moved C2 0.90 mm to (128.3, 103.5)
- moved C1 0.64 mm to (127.6, 72.4)
Connections:
- J2 pad 1: GND -> Net-(J2-Pad1)
- J2 pad 2: Net-(J2-Pad2) -> /9VRET
- J2 pad 3: Net-(J2-Pad3) -> Net-(D1-Pad1)
- J3 pad 1: Net-(J3-Pad1) -> +9V
- J3 pad 2: /9VRET -> GND
- J3 pad 3: +9V -> Net-(J3-Pad3)
- U2 pad 21: Net-(J2-Pad3) -> Net-(U2-Pad21)
- U2 pad 22: Net-(J2-Pad2) -> Net-(U2-Pad22)
- U3 pad 6: Net-(J3-Pad5) -> Net-(C3-Pad1)
- U3 pad 7: Net-(J3-Pad4) -> Net-(C4-Pad1)
Routing:
- net Net-(C4-Pad1): track 0.00 -> 49.0 mm, vias 0 -> 1
- net Net-(C3-Pad1): track 0.00 -> 44.5 mm
- net +9V: track 55.2 -> 29.8 mm
- net Net-(J3-Pad5): track 23.3 -> 0.00 mm, vias 1 -> 0
- net Net-(J3-Pad4): track 22.5 -> 0.00 mm, vias 1 -> 0
- net Net-(D1-Pad1): track 0.00 -> 18.0 mm
- net GND: track 196.1 -> 211.2 mm, vias 4 -> 5
- net Net-(J2-Pad3): track 7.62 -> 0.00 mm
- net Net-(J2-Pad2): track 7.62 -> 0.00 mm
- net Net-(U1-Pad18): track 28.3 -> 32.8 mm, vias 0 -> 1
- net /9VRET: track 13.4 -> 15.1 mm
- net +5V: track 50.9 -> 52.4 mm
- net Net-(J1-Pad2): track 42.8 -> 41.2 mm
- net Net-(Q1-Pad1): track 34.6 -> 36.1 mm
- net Net-(J1-Pad1): track 42.3 -> 43.6 mm
- added copper zone on B.Cu, net GND
- added copper zone on F.Cu, net GND
Other:
- board text added: "G"
- board text added: "S"
- board text removed: "V C GND"
